Commit message: fix(fr-17): 로봇암 A 관절 이름을 URDF 기준 j1~j6으로 통일
FR5 URDF(fr5_gripper.urdf)의 관절 이름이 j1~j6인데 ROS 쪽 URDF, 포즈 설정, Unity RosArmTarget은
joint_1~joint_6을 쓰고 있어 JointState의 name 매칭이 맞지 않았다. 세 곳과 README의 예시 명령을 j1~j6으로 맞췄다.
인터페이스 정의서의 확정이 필요한 항목에서 관절 이름 항목을 완료로 표시.

File: medikit_ws/src/aurix_description/urdf/arm_a.urdf (robot description, URDF)
Before this commit: robot arm_a, 7 links, 6 joints
Joints:
- removed joint joint_1
- removed joint joint_2
- removed joint joint_3
- removed joint joint_4
- removed joint joint_5
- removed joint joint_6
- added joint j1: type revolute, parent base_link, child link_1, origin xyz=0 0 0.2 rpy=0 0 0, axis 0 0 1, limit lower=-3.14159 upper=3.14159 effort=50 velocity=2.0
- added joint j2: type revolute, parent link_1, child link_2, origin xyz=0 0 0.2 rpy=0 0 0, axis 0 1 0, limit lower=-3.14159 upper=3.14159 effort=50 velocity=2.0
- added joint j3: type revolute, parent link_2, child link_3, origin xyz=0 0 0.2 rpy=0 0 0, axis 0 1 0, limit lower=-3.14159 upper=3.14159 effort=50 velocity=2.0
- added joint j4: type revolute, parent link_3, child link_4, origin xyz=0 0 0.2 rpy=0 0 0, axis 0 1 0, limit lower=-3.14159 upper=3.14159 effort=50 velocity=2.0
- added joint j5: type revolute, parent link_4, child link_5, origin xyz=0 0 0.2 rpy=0 0 0, axis 0 0 1, limit lower=-3.14159 upper=3.14159 effort=50 velocity=2.0
- added joint j6: type revolute, parent link_5, child link_6, origin xyz=0 0 0.2 rpy=0 0 0, axis 0 1 0, limit lower=-3.14159 upper=3.14159 effort=50 velocity=2.0
